Commit message: Added slider controller(both python script and launch file

File: install/panda_description/share/panda_description/urdf/arm.xacro (robot description, xacro)
@@ -1,297 +1 @@
-<?xml version="1.0" ?>
-<robot name="panda" xmlns:xacro="http://www.ros.org/wiki/xacro">
-  <!-- World Frame -->
-  <link name="world"/>
-  <!-- Link 0 - Base -->
-  <link name="panda_link0">
-    <visual>
-      <geometry>
-        <mesh filename="package://panda_description/meshes/visual/link0.dae"/>
-      </geometry>
-    </visual>
-    <collision>
-      <geometry>
-        <mesh filename="package://panda_description/meshes/collision/link0.obj"/>
-      </geometry>
-    </collision>
-      <inertial>
-          <origin xyz="0 0 0" rpy="0.0 0.0 0.0"/>
-          <mass value="0.1"/>
-          <inertia ixx="0.1" ixy="0.0" ixz="0.0" iyy="0.1" iyz="0.0" izz="0.1"/>
-      </inertial>
-  </link>
-  <!-- World-Base Joint -->
-  <joint name="virtual_joint" type="fixed">
-    <parent link="world"/>
-    <child link="panda_link0"/>
-    <origin xyz="0.6 0 0.35" rpy="0 0 1.57"/>
-  </joint>
-  <!-- Link 1 -->
-  <link name="panda_link1">
-    <visual>
-      <geometry>
-        <mesh filename="package://panda_description/meshes/visual/link1.dae"/>
-      </geometry>
-    </visual>
-    <collision>
-      <geometry>
-        <mesh filename="package://panda_description/meshes/collision/link1.obj"/>
-      </geometry>
-    </collision>
-        <inertial>
-            <origin xyz="0 0 0" rpy="0.0 0.0 0.0"/>
-            <mass value="0.1"/>
-            <inertia ixx="0.1" ixy="0.0" ixz="0.0" iyy="0.1" iyz="0.0" izz="0.1"/>
-        </inertial>
-  </link>
-  <!-- Joint 1 -->
-  <joint name="panda_joint1" type="revolute">
-    <safety_controller k_position="100.0" k_velocity="40.0" soft_lower_limit="-2.8973" soft_upper_limit="2.8973"/>
-    <origin rpy="0 0 0" xyz="0 0 0.333"/>
-    <parent link="panda_link0"/>
-    <child link="panda_link1"/>
-    <axis xyz="0 0 1"/>
-    <limit effort="30.0" lower="-2.9671" upper="2.9671" velocity="10.0"/>
-  </joint>
-  <!-- Link 2 -->
-  <link name="panda_link2">
-    <visual>
-      <geometry>
-        <mesh filename="package://panda_description/meshes/visual/link2.dae"/>
-      </geometry>
-    </visual>
-    <collision>
-      <geometry>
-        <mesh filename="package://panda_description/meshes/collision/link2.obj"/>
-      </geometry>
-    </collision>
-        <inertial>
-          <origin xyz="0 0 0" rpy="0.0 0.0 0.0"/>
-          <mass value="0.1"/>
-          <inertia ixx="0.1" ixy="0.0" ixz="0.0" iyy="0.1" iyz="0.0" izz="0.1"/>
-      </inertial>
-  </link>
-  <!-- Joint 2 -->
-  <joint name="panda_joint2" type="revolute">
-    <safety_controller k_position="100.0" k_velocity="40.0" soft_lower_limit="-1.7628" soft_upper_limit="1.7628"/>
-    <origin rpy="-1.57079632679 0 0" xyz="0 0 0"/>
-    <parent link="panda_link1"/>
-    <child link="panda_link2"/>
-    <axis xyz="0 0 1"/>
-    <limit effort="30.0" lower="-1.8326" upper="1.8326" velocity="10.0"/>
-  </joint>
-  <!-- Link 3 -->
-  <link name="panda_link3">
-    <visual>
-      <geometry>
-        <mesh filename="package://panda_description/meshes/visual/link3.dae"/>
-      </geometry>
-    </visual>
-    <collision>
-      <geometry>
-        <mesh filename="package://panda_description/meshes/collision/link3.obj"/>
-      </geometry>
-    </collision>
-      <inertial>
-          <origin xyz="0 0 0" rpy="0.0 0.0 0.0"/>
-          <mass value="0.1"/>
-          <inertia ixx="0.1" ixy="0.0" ixz="0.0" iyy="0.1" iyz="0.0" izz="0.1"/>
-      </inertial>
-  </link>
-  <!-- Joint 3 -->
-  <joint name="panda_joint3" type="revolute">
-    <safety_controller k_position="100.0" k_velocity="40.0" soft_lower_limit="-2.8973" soft_upper_limit="2.8973"/>
-    <origin rpy="1.57079632679 0 0" xyz="0 -0.316 0"/>
-    <parent link="panda_link2"/>
-    <child link="panda_link3"/>
-    <axis xyz="0 0 1"/>
-    <limit effort="30.0" lower="-2.9671" upper="2.9671" velocity="10.0"/>
-  </joint>
-  <!-- Link 4 -->
-  <link name="panda_link4">
-    <visual>
-      <geometry>
-        <mesh filename="package://panda_description/meshes/visual/link4.dae"/>
-      </geometry>
-    </visual>
-    <collision>
-      <geometry>
-        <mesh filename="package://panda_description/meshes/collision/link4.obj"/>
-      </geometry>
-    </collision>
-      <inertial>
-          <origin xyz="0 0 0" rpy="0.0 0.0 0.0"/>
-          <mass value="0.1"/>
-          <inertia ixx="0.1" ixy="0.0" ixz="0.0" iyy="0.1" iyz="0.0" izz="0.1"/>
-      </inertial>
-  </link>
-  <!-- Joint 4 -->
-  <joint name="panda_joint4" type="revolute">
-    <safety_controller k_position="100.0" k_velocity="40.0" soft_lower_limit="-3.0718" soft_upper_limit="-0.0698"/>
-    <origin rpy="1.57079632679 0 0" xyz="0.0825 0 0"/>
-    <parent link="panda_link3"/>
-    <child link="panda_link4"/>
-    <axis xyz="0 0 1"/>
-    <limit effort="30.0" lower="-3.1416" upper="0.0" velocity="10.0"/>
-  </joint>
-  <!-- Link 5 -->
-  <link name="panda_link5">
-    <visual>
-      <geometry>
-        <mesh filename="package://panda_description/meshes/visual/link5.dae"/>
-      </geometry>
-    </visual>
-    <collision>
-      <geometry>
-        <mesh filename="package://panda_description/meshes/collision/link5.obj"/>
-      </geometry>
-    </collision>
-      <inertial>
-          <origin xyz="0 0 0" rpy="0.0 0.0 0.0"/>
-          <mass value="0.1"/>
-          <inertia ixx="0.1" ixy="0.0" ixz="0.0" iyy="0.1" iyz="0.0" izz="0.1"/>
-      </inertial>
-  </link>
-  <!-- Joint 5 -->
-  <joint name="panda_joint5" type="revolute">
-    <safety_controller k_position="100.0" k_velocity="40.0" soft_lower_limit="-2.8973" soft_upper_limit="2.8973"/>
-    <origin rpy="-1.57079632679 0 0" xyz="-0.0825 0.384 0"/>
-    <parent link="panda_link4"/>
-    <child link="panda_link5"/>
-    <axis xyz="0 0 1"/>
-    <limit effort="30.0" lower="-2.9671" upper="2.9671" velocity="10.0"/>
-  </joint>
-  <!-- Link 6 -->
-  <link name="panda_link6">
-    <visual>
-      <geometry>
-        <mesh filename="package://panda_description/meshes/visual/link6.dae"/>
-      </geometry>
-    </visual>
-    <collision>
-      <geometry>
-        <mesh filename="package://panda_description/meshes/collision/link6.obj"/>
-      </geometry>
-    </collision>
-      <inertial>
-          <origin xyz="0 0 0" rpy="0.0 0.0 0.0"/>
-          <mass value="0.1"/>
-          <inertia ixx="0.1" ixy="0.0" ixz="0.0" iyy="0.1" iyz="0.0" izz="0.1"/>
-      </inertial>
-  </link>
-  <!-- Joint 6 -->
-  <joint name="panda_joint6" type="revolute">
-    <safety_controller k_position="100.0" k_velocity="40.0" soft_lower_limit="-0.0175" soft_upper_limit="3.7525"/>
-    <origin rpy="1.57079632679 0 0" xyz="0 0 0"/>
-    <parent link="panda_link5"/>
-    <child link="panda_link6"/>
-    <axis xyz="0 0 1"/>
-    <limit effort="30.0" lower="-0.0873" upper="3.8223" velocity="10.0"/>
-  </joint>
-  <!-- Link 7 -->
-  <link name="panda_link7">
-    <visual>
-      <geometry>
-        <mesh filename="package://panda_description/meshes/visual/link7.dae"/>
-      </geometry>
-    </visual>
-    <collision>
-      <geometry>
-        <mesh filename="package://panda_description/meshes/collision/link7.obj"/>
-      </geometry>
-    </collision>
-      <inertial>
-          <origin xyz="0 0 0" rpy="0.0 0.0 0.0"/>
-          <mass value="0.1"/>
-          <inertia ixx="0.1" ixy="0.0" ixz="0.0" iyy="0.1" iyz="0.0" izz="0.1"/>
-      </inertial>
-  </link>
-  <!-- Joint 7 -->
-  <joint name="panda_joint7" type="revolute">
-    <safety_controller k_position="100.0" k_velocity="40.0" soft_lower_limit="-2.8973" soft_upper_limit="2.8973"/>
-    <origin rpy="1.57079632679 0 0" xyz="0.088 0 0"/>
-    <parent link="panda_link6"/>
-    <child link="panda_link7"/>
-    <axis xyz="0 0 1"/>
-    <limit effort="30.0" lower="-2.9671" upper="2.9671" velocity="10.0"/>
-  </joint>
-  <!-- Hand Link -->
-  <link name="panda_hand">
-    <visual>
-      <geometry>
-        <mesh filename="package://panda_description/meshes/visual/hand.dae"/>
-      </geometry>
-    </visual>
-    <collision>
-      <geometry>
-        <mesh filename="package://panda_description/meshes/collision/hand.obj"/>
-      </geometry>
-    </collision>
-      <inertial>
-          <origin xyz="0 0 0" rpy="0.0 0.0 0.0"/>
-          <mass value="0.1"/>
-          <inertia ixx="0.1" ixy="0.0" ixz="0.0" iyy="0.1" iyz="0.0" izz="0.1"/>
-      </inertial>
-  </link>
-  <!-- Hand Joint -->
-  <joint name="panda_hand_joint" type="fixed">
-    <parent link="panda_link7"/>
-    <child link="panda_hand"/>
-    <origin rpy="0 0 -0.785398163397" xyz="0 0 0.106"/>
-  </joint>
-  <!-- Left Finger Link -->
-  <link name="panda_leftfinger">
-    <visual>
-      <geometry>
-        <mesh filename="package://panda_description/meshes/visual/finger.dae"/>
-      </geometry>
-    </visual>
-    <collision>
-      <geometry>
-        <mesh filename="package://panda_description/meshes/collision/finger.obj"/>
-      </geometry>
-    </collision>
-      <inertial>
-          <origin xyz="0 0 0" rpy="0.0 0.0 0.0"/>
-          <mass value="0.1"/>
-          <inertia ixx="0.1" ixy="0.0" ixz="0.0" iyy="0.1" iyz="0.0" izz="0.1"/>
-      </inertial>
-  </link>
-  <!-- Right Finger Link -->
-  <link name="panda_rightfinger">
-    <visual>
-      <origin rpy="0 0 3.14159265359" xyz="0 0 0"/>
-      <geometry>
-        <mesh filename="package://panda_description/meshes/visual/finger.dae"/>
-      </geometry>
-    </visual>
-    <collision>
-      <origin rpy="0 0 3.14159265359" xyz="0 0 0"/>
-      <geometry>
-        <mesh filename="package://panda_description/meshes/collision/finger.obj"/>
-      </geometry>
-    </collision>
-      <inertial>
-          <origin xyz="0 0 0" rpy="0.0 0.0 0.0"/>
-          <mass value="0.1"/>
-          <inertia ixx="0.1" ixy="0.0" ixz="0.0" iyy="0.1" iyz="0.0" izz="0.1"/>
-      </inertial>
-  </link>
-  <!-- Finger Joint 1 -->
-  <joint name="panda_finger_joint1" type="prismatic">
-    <parent link="panda_hand"/>
-    <child link="panda_leftfinger"/>
-    <origin rpy="0 0 0" xyz="0 0 0.0584"/>
-    <axis xyz="0 1 0"/>
-    <limit effort="30.0" lower="0.0" upper="0.04" velocity="10.0"/>
-  </joint>
-  <!-- Finger Joint 2 -->
-  <joint name="panda_finger_joint2" type="prismatic">
-    <parent link="panda_hand"/>
-    <child link="panda_rightfinger"/>
-    <origin rpy="0 0 0" xyz="0 0 0.0584"/>
-    <axis xyz="0 -1 0"/>
-    <limit effort="30.0" lower="0.0" upper="0.04" velocity="10.0"/>
-    <!-- <mimic joint="panda_finger_joint1" multiplier="-1"/> -->
-  </joint>
-</robot>
+/home/sreeharischandra/panda_ws/src/panda_description/urdf/arm.xacro

File: install/panda_description/share/panda_description/urdf/gazebo.xacro (robot description, xacro)
@@ -1,91 +1 @@
-<?xml version="1.0"?>
-<robot xmlns:xacro="http://www.ros.org/wiki/xacro" name="panda">
-  <xacro:property name="PI" value="3.14159265359" />
-  <ros2_control name="RobotSystem" type="system">
-    <!-- ros2_control Gazebo -->
-    <!-- ROS 2 Humble -->
-    <xacro:if value="$(arg is_ignition)">
-      <hardware>
-        <plugin>ign_ros2_control/IgnitionSystem</plugin>
-      </hardware>
-    </xacro:if>
-    <!-- ROS 2 Iron or above -->
-    <xacro:unless value="$(arg is_ignition)">
-      <hardware>
-        <plugin>gz_ros2_control/GazeboSimSystem</plugin>
-      </hardware>
-    </xacro:unless>
-    <!-- Joint 1 -->
-    <joint name="panda_joint1">
-      <command_interface name="position">
-        <param name="min">-2.9671</param>
-        <param name="max">2.9671</param>
-      </command_interface>
-      <state_interface name="position"/>
-    </joint>
-    <!-- Joint 2 -->
-    <joint name="panda_joint2">
-      <command_interface name="position">
-        <param name="min">-1.8326</param>
-        <param name="max">1.8326</param>
-      </command_interface>
-      <state_interface name="position"/>
-    </joint>
-    <!-- Joint 3 -->
-    <joint name="panda_joint3">
-      <command_interface name="position">
-        <param name="min">-2.9671</param>
-        <param name="max">2.9671</param>
-      </command_interface>
-      <state_interface name="position"/>
-    </joint>
-    <!-- Joint 4 -->
-    <joint name="panda_joint4">
-      <command_interface name="position">
-        <param name="min">-3.1416</param>
-        <param name="max">0.0</param>
-      </command_interface>
-      <state_interface name="position"/>
-    </joint>
-    <!-- Joint 5 -->
-    <joint name="panda_joint5">
-      <command_interface name="position">
-        <param name="min">-2.9671</param>
-        <param name="max">2.9671</param>
-      </command_interface>
-      <state_interface name="position"/>
-    </joint>
-    <!-- Joint 6 -->
-    <joint name="panda_joint6">
-      <command_interface name="position">
-        <param name="min">-0.0873</param>
-        <param name="max">3.8223</param>
-      </command_interface>
-      <state_interface name="position"/>
-    </joint>
-    <!-- Joint 7 -->
-    <joint name="panda_joint7">
-      <command_interface name="position">
-        <param name="min">-2.9671</param>
-        <param name="max">2.9671</param>
-      </command_interface>
-      <state_interface name="position"/>
-    </joint>
-    <!-- Gripper Finger Joint 1 -->
-    <joint name="panda_finger_joint1">
-      <command_interface name="position">
-        <param name="min">0.0</param>
-        <param name="max">0.04</param>
-      </command_interface>
-      <state_interface name="position"/>
-    </joint>
-    <!-- Gripper Finger Joint 2 (Mimics Joint 1) -->
-    <joint name="panda_finger_joint2">
-      <command_interface name="position">
-        <param name="min">0.0</param>
-        <param name="max">0.04</param>
-      </command_interface>
-      <state_interface name="position"/>
-    </joint>
-  </ros2_control>
-</robot>
+/home/sreeharischandra/panda_ws/src/panda_description/urdf/gazebo.xacro

File: install/panda_description/share/panda_description/urdf/panda.urdf.xacro (robot description, xacro)
@@ -1,5 +1 @@
-<?xml version="1.0"?>
-<robot name="panda" xmlns:xacro="http://www.ros.org/wiki/xacro">
-  <xacro:include filename="$(find panda_description)/urdf/arm.xacro" />
-  <xacro:include filename="$(find panda_description)/urdf/gazebo.xacro" />
-</robot>
+/home/sreeharischandra/panda_ws/src/panda_description/urdf/panda.urdf.xacro

File: install/panda_description/share/panda_description/urdf/ros2control.xacro (robot description, xacro)
@@ -1,24 +1 @@
-<?xml version="1.0"?>
-<robot xmlns:xacro="http://www.ros.org/wiki/xacro" name="panda">
-  <!-- ROS 2 Control -->
-  <!-- ROS 2 Humble -->
-  <gazebo>
-    <xacro:if value="$(arg is_ignition)">
-      <plugin filename="ign_ros2_control-system" name="ign_ros2_control::IgnitionROS2ControlPlugin">
-        <parameters>$(find panda_controller)/config/panda_controllers.yaml</parameters>
-      </plugin>
-      <plugin filename="ignition-gazebo-sensors-system" name="ignition::gazebo::systems::Sensors">
-        <render_engine>ogre2</render_engine>
-      </plugin>
-    </xacro:if>
-    <!-- ROS 2 Iron or above -->
-    <xacro:unless value="$(arg is_ignition)">
-      <plugin filename="gz_ros2_control-system" name="gz_ros2_control::GazeboSimROS2ControlPlugin">
-        <parameters>$(find panda_controller)/config/panda_controllers.yaml</parameters>
-      </plugin>
-      <plugin filename="gz-sim-sensors-system" name="gz::sim::systems::Sensors">
-        <render_engine>ogre2</render_engine>
-      </plugin>
-    </xacro:unless>
-  </gazebo>
-</robot>
+/home/sreeharischandra/panda_ws/src/panda_description/urdf/ros2control.xacro
